Commit message: Modified joint publish rate and velocity limits

File: baxter_gazebo/urdf/baxter_base/baxter_base.urdf.xacro (robot description, xacro)
@@ -517,5 +517,5 @@
     <parent link="right_arm_mount"/>
     <child link="right_upper_shoulder"/>
-    <limit effort="50.0" lower="-1.70167993878" upper="1.70167993878" velocity="1.5"/>
+    <limit effort="50.0" lower="-1.70167993878" upper="1.70167993878" velocity="2.0"/>
     <dynamics damping="0.7" friction="0.0"/>
   </joint>
@@ -525,5 +525,5 @@
     <parent link="right_upper_shoulder"/>
     <child link="right_lower_shoulder"/>
-    <limit effort="50.0" lower="-2.147" upper="1.047" velocity="1.5"/>
+    <limit effort="50.0" lower="-2.147" upper="1.047" velocity="2.0"/>
     <dynamics damping="0.7" friction="0.0"/>
   </joint>
@@ -533,5 +533,5 @@
     <parent link="right_lower_shoulder"/>
     <child link="right_upper_elbow"/>
-    <limit effort="50.0" lower="-3.05417993878" upper="3.05417993878" velocity="1.5"/>
+    <limit effort="50.0" lower="-3.05417993878" upper="3.05417993878" velocity="2.0"/>
     <dynamics damping="0.7" friction="0.0"/>
   </joint>
@@ -547,5 +547,5 @@
     <parent link="right_upper_elbow"/>
     <child link="right_lower_elbow"/>
-    <limit effort="50.0" lower="-0.05" upper="2.618" velocity="1.5"/>
+    <limit effort="50.0" lower="-0.05" upper="2.618" velocity="2.0"/>
     <dynamics damping="0.7" friction="0.0"/>
   </joint>
@@ -885,5 +885,5 @@
     <parent link="left_arm_mount"/>
     <child link="left_upper_shoulder"/>
-    <limit effort="50.0" lower="-1.70167993878" upper="1.70167993878" velocity="1.5"/>
+    <limit effort="50.0" lower="-1.70167993878" upper="1.70167993878" velocity="2.0"/>
     <dynamics damping="0.7" friction="0.0"/>
   </joint>
@@ -893,5 +893,5 @@
     <parent link="left_upper_shoulder"/>
     <child link="left_lower_shoulder"/>
-    <limit effort="50.0" lower="-2.147" upper="1.047" velocity="1.5"/>
+    <limit effort="50.0" lower="-2.147" upper="1.047" velocity="2.0"/>
     <dynamics damping="0.7" friction="0.0"/>
   </joint>
@@ -901,5 +901,5 @@
     <parent link="left_lower_shoulder"/>
     <child link="left_upper_elbow"/>
-    <limit effort="50.0" lower="-3.05417993878" upper="3.05417993878" velocity="1.5"/>
+    <limit effort="50.0" lower="-3.05417993878" upper="3.05417993878" velocity="2.0"/>
     <dynamics damping="0.7" friction="0.0"/>
   </joint>
@@ -915,5 +915,5 @@
     <parent link="left_upper_elbow"/>
     <child link="left_lower_elbow"/>
-    <limit effort="50.0" lower="-0.05" upper="2.618" velocity="1.5"/>
+    <limit effort="50.0" lower="-0.05" upper="2.618" velocity="2.0"/>
     <dynamics damping="0.7" friction="0.0"/>
   </joint>
