Commit message: fixed bugs and update to noetic

File: baxter_gazebo/urdf/baxter.urdf (robot description, URDF)
Before this commit: robot baxter, 58 links, 57 joints
Links:
- link head: geometry collision sphere radius=0.001; visual mesh filename=package://baxter_gazebo/meshes/head/H0.dae
- link left_lower_elbow: geometry collision cylinder length=0.10 radius=0.06; visual mesh filename=package://baxter_gazebo/meshes/lower_elbow/E1.dae
- link left_lower_forearm: geometry collision cylinder length=0.10 radius=0.06; visual mesh filename=package://baxter_gazebo/meshes/lower_forearm/W1.dae
- link left_lower_shoulder: geometry collision cylinder length=0.12 radius=0.06; visual mesh filename=package://baxter_gazebo/meshes/lower_shoulder/S1.dae
- link left_upper_elbow: geometry collision cylinder length=0.107 radius=0.06; visual mesh filename=package://baxter_gazebo/meshes/upper_elbow/E0.dae
- link left_upper_forearm: geometry collision cylinder length=0.088 radius=0.06; visual mesh filename=package://baxter_gazebo/meshes/upper_forearm/W0.dae
- link left_upper_shoulder: geometry collision cylinder length=0.2722 radius=0.06; visual mesh filename=package://baxter_gazebo/meshes/upper_shoulder/S0.dae
- link left_wrist: geometry collision cylinder length=0.165 radius=0.06; visual mesh filename=package://baxter_gazebo/meshes/wrist/W2.dae
- link pedestal: geometry collision mesh filename=package://baxter_gazebo/meshes/base/pedestal_link_collision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; visual mesh filename=package://baxter_gazebo/meshes/base/PEDESTAL.dae
- link right_lower_elbow: geometry collision cylinder length=0.10 radius=0.06; visual mesh filename=package://baxter_gazebo/meshes/lower_elbow/E1.dae
- link right_lower_forearm: geometry collision cylinder length=0.10 radius=0.06; visual mesh filename=package://baxter_gazebo/meshes/lower_forearm/W1.dae
- link right_lower_shoulder: geometry collision cylinder length=0.12 radius=0.06; visual mesh filename=package://baxter_gazebo/meshes/lower_shoulder/S1.dae
- link right_upper_elbow: geometry collision cylinder length=0.107 radius=0.06; visual mesh filename=package://baxter_gazebo/meshes/upper_elbow/E0.dae
- link right_upper_forearm: geometry collision cylinder length=0.088 radius=0.06; visual mesh filename=package://baxter_gazebo/meshes/upper_forearm/W0.dae
- link right_upper_shoulder: geometry collision cylinder length=0.2722 radius=0.06; visual mesh filename=package://baxter_gazebo/meshes/upper_shoulder/S0.dae
- link right_wrist: geometry collision cylinder length=0.165 radius=0.06; visual mesh filename=package://baxter_gazebo/meshes/wrist/W2.dae
- link screen: geometry collision sphere radius=0.001; visual mesh filename=package://baxter_gazebo/meshes/head/H1.dae
- link torso: geometry collision mesh filename=package://baxter_gazebo/meshes/torso/base_link_collision.dae; visual mesh filename=package://baxter_gazebo/meshes/torso/base_link.dae

File: baxter_gazebo/urdf/baxter_base/baxter_base.urdf.xacro (robot description, xacro)
@@ -12,5 +12,5 @@
       <origin rpy="0 0 0" xyz="0 0 0"/>
       <geometry>
-        <mesh filename="package://baxter_gazebo/meshes/torso/base_link.DAE"/>
+        <mesh filename="package://baxter_gazebo/meshes/torso/base_link.dae"/>
       </geometry>
       <material name="darkgray">
@@ -21,5 +21,5 @@
       <origin rpy="0 0 0" xyz="0 0 0"/>
       <geometry>
-        <mesh filename="package://baxter_gazebo/meshes/torso/base_link_collision.DAE"/>
+        <mesh filename="package://baxter_gazebo/meshes/torso/base_link_collision.dae"/>
       </geometry>
     </collision>
@@ -48,5 +48,5 @@
       <origin rpy="0 0 0" xyz="0 0 .00953"/>
       <geometry>
-        <mesh filename="package://baxter_gazebo/meshes/head/H0.DAE"/>
+        <mesh filename="package://baxter_gazebo/meshes/head/H0.dae"/>
       </geometry>
       <material name="darkgray">
@@ -92,5 +92,5 @@
       <origin rpy="0 -1.57079632679 0" xyz="0 -.00953 -.0347"/>
       <geometry>
-        <mesh filename="package://baxter_gazebo/meshes/head/H1.DAE"/>
+        <mesh filename="package://baxter_gazebo/meshes/head/H1.dae"/>
       </geometry>
       <material name="darkred">
@@ -256,5 +256,5 @@
       <origin rpy="0 0 0" xyz="0 0 0"/>
       <geometry>
-        <mesh filename="package://baxter_gazebo/meshes/upper_shoulder/S0.DAE"/>
+        <mesh filename="package://baxter_gazebo/meshes/upper_shoulder/S0.dae"/>
       </geometry>
       <material name="darkred">
@@ -278,5 +278,5 @@
       <origin rpy="0 0 0" xyz="0 0 0"/>
       <geometry>
-        <mesh filename="package://baxter_gazebo/meshes/lower_shoulder/S1.DAE"/>
+        <mesh filename="package://baxter_gazebo/meshes/lower_shoulder/S1.dae"/>
       </geometry>
       <material name="darkred">
@@ -300,5 +300,5 @@
       <origin rpy="0 0 0" xyz="0 0 0"/>
       <geometry>
-        <mesh filename="package://baxter_gazebo/meshes/upper_elbow/E0.DAE"/>
+        <mesh filename="package://baxter_gazebo/meshes/upper_elbow/E0.dae"/>
       </geometry>
       <material name="darkred">
@@ -335,5 +335,5 @@
       <origin rpy="0 0 0" xyz="0 0 0"/>
       <geometry>
-        <mesh filename="package://baxter_gazebo/meshes/lower_elbow/E1.DAE"/>
+        <mesh filename="package://baxter_gazebo/meshes/lower_elbow/E1.dae"/>
       </geometry>
       <material name="darkred">
@@ -357,5 +357,5 @@
       <origin rpy="0 0 0" xyz="0 0 0"/>
       <geometry>
-        <mesh filename="package://baxter_gazebo/meshes/upper_forearm/W0.DAE"/>
+        <mesh filename="package://baxter_gazebo/meshes/upper_forearm/W0.dae"/>
       </geometry>
       <material name="darkred">
@@ -399,5 +399,5 @@
       <origin rpy="0 0 0" xyz="0 0 0"/>
       <geometry>
-        <mesh filename="package://baxter_gazebo/meshes/lower_forearm/W1.DAE"/>
+        <mesh filename="package://baxter_gazebo/meshes/lower_forearm/W1.dae"/>
       </geometry>
       <material name="darkred">
@@ -421,5 +421,5 @@
       <origin rpy="0 0 0" xyz="0 0 0"/>
       <geometry>
-        <mesh filename="package://baxter_gazebo/meshes/wrist/W2.DAE"/>
+        <mesh filename="package://baxter_gazebo/meshes/wrist/W2.dae"/>
       </geometry>
       <material name="lightgrey">
@@ -624,5 +624,5 @@
       <origin rpy="0 0 0" xyz="0 0 0"/>
       <geometry>
-        <mesh filename="package://baxter_gazebo/meshes/upper_shoulder/S0.DAE"/>
+        <mesh filename="package://baxter_gazebo/meshes/upper_shoulder/S0.dae"/>
       </geometry>
       <material name="darkred">
@@ -646,5 +646,5 @@
       <origin rpy="0 0 0" xyz="0 0 0"/>
       <geometry>
-        <mesh filename="package://baxter_gazebo/meshes/lower_shoulder/S1.DAE"/>
+        <mesh filename="package://baxter_gazebo/meshes/lower_shoulder/S1.dae"/>
       </geometry>
       <material name="darkred">
@@ -668,5 +668,5 @@
       <origin rpy="0 0 0" xyz="0 0 0"/>
       <geometry>
-        <mesh filename="package://baxter_gazebo/meshes/upper_elbow/E0.DAE"/>
+        <mesh filename="package://baxter_gazebo/meshes/upper_elbow/E0.dae"/>
       </geometry>
       <material name="darkred">
@@ -703,5 +703,5 @@
       <origin rpy="0 0 0" xyz="0 0 0"/>
       <geometry>
-        <mesh filename="package://baxter_gazebo/meshes/lower_elbow/E1.DAE"/>
+        <mesh filename="package://baxter_gazebo/meshes/lower_elbow/E1.dae"/>
       </geometry>
       <material name="darkred">
@@ -725,5 +725,5 @@
       <origin rpy="0 0 0" xyz="0 0 0"/>
       <geometry>
-        <mesh filename="package://baxter_gazebo/meshes/upper_forearm/W0.DAE"/>
+        <mesh filename="package://baxter_gazebo/meshes/upper_forearm/W0.dae"/>
       </geometry>
       <material name="darkred">
@@ -767,5 +767,5 @@
       <origin rpy="0 0 0" xyz="0 0 0"/>
       <geometry>
-        <mesh filename="package://baxter_gazebo/meshes/lower_forearm/W1.DAE"/>
+        <mesh filename="package://baxter_gazebo/meshes/lower_forearm/W1.dae"/>
       </geometry>
       <material name="darkred">
@@ -789,5 +789,5 @@
       <origin rpy="0 0 0" xyz="0 0 0"/>
       <geometry>
-        <mesh filename="package://baxter_gazebo/meshes/wrist/W2.DAE"/>
+        <mesh filename="package://baxter_gazebo/meshes/wrist/W2.dae"/>
       </geometry>
       <material name="lightgrey">

File: baxter_gazebo/urdf/pedestal/pedestal.xacro (robot description, xacro)
@@ -7,5 +7,5 @@
       <origin rpy="0 0 0" xyz="0 0 0"/>
       <geometry>
-        <mesh filename="package://baxter_gazebo/meshes/base/PEDESTAL.DAE"/>
+        <mesh filename="package://baxter_gazebo/meshes/base/PEDESTAL.dae"/>
       </geometry>
       <material name="darkgray">
@@ -16,5 +16,5 @@
       <origin rpy="0 0 0" xyz="0 0 0"/>
       <geometry>
-        <mesh filename="package://baxter_gazebo/meshes/base/pedestal_link_collision.DAE"/>
+        <mesh filename="package://baxter_gazebo/meshes/base/pedestal_link_collision.dae"/>
       </geometry>
     </collision>
